Commit message: u

File: dql_robot/urdf/ABot.urdf.xacro (robot description, xacro)
@@ -27,5 +27,5 @@
   </collision>
   </link>
-  <link name="camera_link">
+  <link name="camera_link1">
     <collision>
       <origin xyz="0 0 0" rpy="0 0 0"/>
@@ -47,9 +47,35 @@
     </inertial>
   </link>
-  <joint name="camera_joint" type="fixed">
+  <link name="camera_link2">
+    <collision>
+      <origin xyz="0 0 0" rpy="0 0 0"/>
+      <geometry>
+    <box size="0.01 0.01 0.01"/>
+      </geometry>
+    </collision>
+    <visual>
+      <origin xyz="0 0 0" rpy="0 0 0"/>
+      <geometry>
+    <box size="0.01 0.01 0.01"/>
+      </geometry>
+      <material name="red"/>
+    </visual>
+    <inertial>
+      <mass value="1e-5" />
+      <origin xyz="0 0 0" rpy="0 0 0"/>
+      <inertia ixx="1e-6" ixy="0" ixz="0" iyy="1e-6" iyz="0" izz="1e-6" />
+    </inertial>
+  </link>
+  <joint name="camera_joint1" type="fixed">
     <axis xyz="0 1 0" />
     <origin xyz="0.23 0 0.25" rpy="0 0 0"/>
     <parent link="base_link"/>
-    <child link="camera_link"/>
+    <child link="camera_link1"/>
+  </joint>
+  <joint name="camera_joint2" type="fixed">
+    <axis xyz="0 1 0" />
+    <origin xyz="-0.23 0 0.25" rpy="0 0 3.1415"/>
+    <parent link="base_link"/>
+    <child link="camera_link2"/>
   </joint>
   <link name="box">
@@ -286,6 +312,6 @@
   </plugin>
 </gazebo>
-<!-- camera -->
-  <gazebo reference="camera_link">
+<!-- front camera -->
+  <gazebo reference="camera_link1">
     <sensor type="camera" name="camera1">
       <update_rate>30.0</update_rate>
@@ -313,8 +339,8 @@
         <alwaysOn>true</alwaysOn>
         <updateRate>0.0</updateRate>
-        <cameraName>/camera</cameraName>
+        <cameraName>/front_camera</cameraName>
         <imageTopicName>image_raw</imageTopicName>
         <cameraInfoTopicName>camera_info</cameraInfoTopicName>
-        <frameName>camera_link</frameName>
+        <frameName>camera_link1</frameName>
         <hackBaseline>0.07</hackBaseline>
         <distortionK1>0.0</distortionK1>
@@ -326,4 +352,45 @@
     </sensor>
   </gazebo>
-  <xacro:property name="camera_link" value="0.05" /> <!-- Size of square 'camera' box -->
+	<!-- back camera -->
+  <gazebo reference="camera_link2">
+    <sensor type="camera" name="camera2">
+      <update_rate>30.0</update_rate>
+      <camera name="head">
+        <horizontal_fov>1.3962634</horizontal_fov>
+        <image>
+          <width>640</width>
+          <height>480</height>
+          <format>R8G8B8</format>
+        </image>
+        <clip>
+          <near>0.02</near>
+          <far>300</far>
+        </clip>
+        <noise>
+          <type>gaussian</type>
+          <!-- Noise is sampled independently per pixel on each frame.
+               That pixel's noise value is added to each of its color
+               channels, which at that point lie in the range [0,1]. -->
+          <mean>0.0</mean>
+          <stddev>0.007</stddev>
+        </noise>
+      </camera>
+      <plugin name="camera_controller" filename="libgazebo_ros_camera.so">
+        <alwaysOn>true</alwaysOn>
+        <updateRate>0.0</updateRate>
+        <cameraName>/back_camera</cameraName>
+        <imageTopicName>image_raw</imageTopicName>
+        <cameraInfoTopicName>camera_info</cameraInfoTopicName>
+        <frameName>camera_link2</frameName>
+        <hackBaseline>0.07</hackBaseline>
+        <distortionK1>0.0</distortionK1>
+        <distortionK2>0.0</distortionK2>
+        <distortionK3>0.0</distortionK3>
+        <distortionT1>0.0</distortionT1>
+        <distortionT2>0.0</distortionT2>
+      </plugin>
+    </sensor>
+  </gazebo>
+  <xacro:property name="camera_link1" value="0.05" /> <!-- Size of square 'camera' box -->
+  <xacro:property name="camera_link2" value="0.05" /> <!-- Size of square 'camera' box -->
 </robot>

Commit message: u

File: dql_robot/urdf/ABot.urdf.xacro (robot description, xacro)
@@ -69,5 +69,5 @@
   <joint name="camera_joint1" type="fixed">
     <axis xyz="0 1 0" />
-    <origin xyz="0.23 0 0.25" rpy="0 0 0"/>
+    <origin xyz="0.2 0 0.25" rpy="0 0 0"/>
     <parent link="base_link"/>
     <child link="camera_link1"/>
@@ -75,5 +75,5 @@
   <joint name="camera_joint2" type="fixed">
     <axis xyz="0 1 0" />
-    <origin xyz="-0.23 0 0.25" rpy="0 0 3.1415"/>
+    <origin xyz="-0.2 0 0.25" rpy="0 0 3.1415"/>
     <parent link="base_link"/>
     <child link="camera_link2"/>
@@ -183,5 +183,5 @@
     </joint>
   </transmission>
-  <link name="back_wheel">
+  <link name="back_wheel1">
   <inertial>
     <origin rpy="1.5707963267948966 0 0" xyz="0 0 0" />
@@ -204,18 +204,54 @@
         <friction>
           <ode>
-            <mu>0.01</mu>
-            <mu2>0.01</mu2>
+            <mu>0.0001</mu>
+            <mu2>0.0001</mu2>
           </ode>
         </friction>
       </surface>
   </link>
-  <gazebo reference="back_wheel">
+  <link name="back_wheel2">
+  <inertial>
+    <origin rpy="1.5707963267948966 0 0" xyz="0 0 0" />
+    <mass value="0.1" />
+    <inertia  ixx="0.01" ixy="0.0"  ixz="0.0"  iyy="0.01"  iyz="0.0"  izz="0.01" />
+  </inertial>
+  <visual>
+    <origin rpy="1.5707963267948966 0 0" xyz="0 0 0"/>
+    <geometry>
+      <sphere length="0.1" radius="0.025"/>
+    </geometry>
+  </visual>
+  <collision>
+    <origin rpy="1.5707963267948966 0 0" xyz="0 0 0"/>
+    <geometry>
+      <sphere length="0.1" radius="0.025"/>
+    </geometry>
+  </collision>
+      <surface>
+        <friction>
+          <ode>
+            <mu>0.0001</mu>
+            <mu2>0.0001</mu2>
+          </ode>
+        </friction>
+      </surface>
+  </link>
+  <gazebo reference="back_wheel1">
     <material>Gazebo/White</material>
   </gazebo>
-  <joint name="base_link_back_wheel" type="continuous">
-    <parent link="base_link"/>
-    <child link="back_wheel"/>
+  <gazebo reference="back_wheel2">
+    <material>Gazebo/White</material>
+  </gazebo>
+  <joint name="base_link_back_wheel1" type="continuous">
+    <parent link="base_link"/>
+    <child link="back_wheel1"/>
     <axis xyz="0 1 1"/>
-    <origin xyz="-0.15 0 0.025"/>
+    <origin xyz="-0.15 0.1 0.025"/>
+  </joint>
+  <joint name="base_link_back_wheel2" type="continuous">
+    <parent link="base_link"/>
+    <child link="back_wheel2"/>
+    <axis xyz="0 1 1"/>
+    <origin xyz="-0.15 -0.1 0.025"/>
   </joint>
   <!--link name="right_back_wheel">
@@ -303,5 +339,5 @@
     <wheelSeparation>0.35</wheelSeparation>
     <wheelDiameter>0.15</wheelDiameter>
-    <torque>1.41</torque>
+    <torque>0.41</torque>
     <commandTopic>cmd_vel</commandTopic>
     <odometryTopic>odom</odometryTopic>

Commit message: u

File: dql_robot/urdf/ABot.urdf.xacro (robot description, xacro)
@@ -11,6 +11,6 @@
   <inertial>
     <origin xyz="0 0 0.125" />
-    <mass value="5" />
-    <inertia  ixx="0.1" ixy="0.0"  ixz="0.0"  iyy="0.1"  iyz="0.0"  izz="0.1" />
+    <mass value="15" />
+    <inertia  ixx="1.1" ixy="0.0"  ixz="0.0"  iyy="1.1"  iyz="0.0"  izz="1.1" />
   </inertial>
   <visual>
@@ -339,5 +339,5 @@
     <wheelSeparation>0.35</wheelSeparation>
     <wheelDiameter>0.15</wheelDiameter>
-    <torque>0.41</torque>
+    <torque>1.41</torque>
     <commandTopic>cmd_vel</commandTopic>
     <odometryTopic>odom</odometryTopic>
