Commit message: u

File: dql_robot/urdf/predator.urdf.xacro (robot description, xacro)
@@ -116,17 +116,14 @@
     <origin rpy="1.5707963267948966 0 0" xyz="0 0 0"/>
     <geometry>
-      <cylinder length="0.05" radius="0.075"/>
-    </geometry>
-  </visual>
-  <collision>
-    <origin rpy="1.5707963267948966 0 0" xyz="0 0 0"/>
-    <geometry>
-      <cylinder length="0.05" radius="0.075"/>
-    </geometry>
-  </collision>
-  </link>
-  <gazebo reference="right_wheel">
-    <material>Gazebo/Black</material>
-  </gazebo>
+      <cylinder length="0.01" radius="0.075"/>
+    </geometry>
+  </visual>
+  <collision>
+    <origin rpy="1.5707963267948966 0 0" xyz="0 0 0"/>
+    <geometry>
+      <cylinder length="0.01" radius="0.075"/>
+    </geometry>
+  </collision>
+  </link>
   <joint name="base_link_right_wheel" type="continuous">
     <parent link="base_link"/>
@@ -154,17 +151,14 @@
     <origin rpy="1.5707963267948966 0 0" xyz="0 0 0"/>
     <geometry>
-      <cylinder length="0.05" radius="0.075"/>
-    </geometry>
-  </visual>
-  <collision>
-    <origin rpy="1.5707963267948966 0 0" xyz="0 0 0"/>
-    <geometry>
-      <cylinder length="0.05" radius="0.075"/>
-    </geometry>
-  </collision>
-  </link>
-  <gazebo reference="left_wheel">
-    <material>Gazebo/Black</material>
-  </gazebo>
+      <cylinder length="0.01" radius="0.075"/>
+    </geometry>
+  </visual>
+  <collision>
+    <origin rpy="1.5707963267948966 0 0" xyz="0 0 0"/>
+    <geometry>
+      <cylinder length="0.01" radius="0.075"/>
+    </geometry>
+  </collision>
+  </link>
   <joint name="base_link_left_wheel" type="continuous">
     <parent link="base_link"/>
@@ -204,6 +198,6 @@
         <friction>
           <ode>
-            <mu>0.0001</mu>
-            <mu2>0.0001</mu2>
+            <mu>0.0</mu>
+            <mu2>0.0</mu2>
           </ode>
         </friction>
@@ -231,16 +225,10 @@
         <friction>
           <ode>
-            <mu>0.0001</mu>
-            <mu2>0.0001</mu2>
+            <mu>0.0</mu>
+            <mu2>0.0</mu2>
           </ode>
         </friction>
       </surface>
   </link>
-  <gazebo reference="back_wheel1">
-    <material>Gazebo/White</material>
-  </gazebo>
-  <gazebo reference="back_wheel2">
-    <material>Gazebo/White</material>
-  </gazebo>
   <joint name="base_link_back_wheel1" type="continuous">
     <parent link="base_link"/>
@@ -331,4 +319,24 @@
     </joint>
   </transmission-->
+ <gazebo reference="back_wheel1">
+    <mu1>0.0</mu1>
+    <mu2>0.0</mu2>
+    <material>Gazebo/Black</material>
+  </gazebo>
+  <gazebo reference="back_wheel2">
+    <mu1>0.0</mu1>
+    <mu2>0.0</mu2>
+    <material>Gazebo/Black</material>
+  </gazebo>
+<gazebo reference="left_wheel">
+    <mu1>1.0</mu1>
+    <mu2>0.5</mu2>
+    <material>Gazebo/Black</material>
+  </gazebo>
+  <gazebo reference="right_wheel">
+    <mu1>1.0</mu1>
+    <mu2>0.5</mu2>
+    <material>Gazebo/Black</material>
+  </gazebo>
 <gazebo>
   <plugin name="differential_drive_controller" filename="libgazebo_ros_diff_drive.so">
@@ -337,7 +345,7 @@
     <leftJoint>base_link_left_wheel</leftJoint>
     <rightJoint>base_link_right_wheel</rightJoint>
-    <wheelSeparation>0.35</wheelSeparation>
+    <wheelSeparation>0.3</wheelSeparation>
     <wheelDiameter>0.15</wheelDiameter>
-    <torque>1.41</torque>
+    <torque>10</torque>
     <commandTopic>cmd_vel</commandTopic>
     <odometryTopic>odom</odometryTopic>
@@ -353,5 +361,5 @@
       <update_rate>30.0</update_rate>
       <camera name="head">
-        <horizontal_fov>1.3962634</horizontal_fov>
+        <horizontal_fov>1.8</horizontal_fov>
         <image>
           <width>640</width>
@@ -393,5 +401,5 @@
       <update_rate>30.0</update_rate>
       <camera name="head">
-        <horizontal_fov>1.3962634</horizontal_fov>
+        <horizontal_fov>0.7</horizontal_fov>
         <image>
           <width>640</width>

File: dql_robot/urdf/prey.urdf.xacro (robot description, xacro)
@@ -116,17 +116,14 @@
     <origin rpy="1.5707963267948966 0 0" xyz="0 0 0"/>
     <geometry>
-      <cylinder length="0.05" radius="0.075"/>
-    </geometry>
-  </visual>
-  <collision>
-    <origin rpy="1.5707963267948966 0 0" xyz="0 0 0"/>
-    <geometry>
-      <cylinder length="0.05" radius="0.075"/>
-    </geometry>
-  </collision>
-  </link>
-  <gazebo reference="right_wheel">
-    <material>Gazebo/Black</material>
-  </gazebo>
+      <cylinder length="0.01" radius="0.075"/>
+    </geometry>
+  </visual>
+  <collision>
+    <origin rpy="1.5707963267948966 0 0" xyz="0 0 0"/>
+    <geometry>
+      <cylinder length="0.01" radius="0.075"/>
+    </geometry>
+  </collision>
+  </link>
   <joint name="base_link_right_wheel" type="continuous">
     <parent link="base_link"/>
@@ -154,17 +151,14 @@
     <origin rpy="1.5707963267948966 0 0" xyz="0 0 0"/>
     <geometry>
-      <cylinder length="0.05" radius="0.075"/>
-    </geometry>
-  </visual>
-  <collision>
-    <origin rpy="1.5707963267948966 0 0" xyz="0 0 0"/>
-    <geometry>
-      <cylinder length="0.05" radius="0.075"/>
-    </geometry>
-  </collision>
-  </link>
-  <gazebo reference="left_wheel">
-    <material>Gazebo/Black</material>
-  </gazebo>
+      <cylinder length="0.01" radius="0.075"/>
+    </geometry>
+  </visual>
+  <collision>
+    <origin rpy="1.5707963267948966 0 0" xyz="0 0 0"/>
+    <geometry>
+      <cylinder length="0.01" radius="0.075"/>
+    </geometry>
+  </collision>
+  </link>
   <joint name="base_link_left_wheel" type="continuous">
     <parent link="base_link"/>
@@ -204,6 +198,6 @@
         <friction>
           <ode>
-            <mu>0.0001</mu>
-            <mu2>0.0001</mu2>
+            <mu>0.0</mu>
+            <mu2>0.0</mu2>
           </ode>
         </friction>
@@ -231,6 +225,6 @@
         <friction>
           <ode>
-            <mu>0.0001</mu>
-            <mu2>0.0001</mu2>
+            <mu>0.0</mu>
+            <mu2>0.0</mu2>
           </ode>
         </friction>
@@ -331,4 +325,24 @@
     </joint>
   </transmission-->
+ <gazebo reference="back_wheel1">
+    <mu1>0.0</mu1>
+    <mu2>0.0</mu2>
+    <material>Gazebo/Black</material>
+  </gazebo>
+  <gazebo reference="back_wheel2">
+    <mu1>0.0</mu1>
+    <mu2>0.0</mu2>
+    <material>Gazebo/Black</material>
+  </gazebo>
+<gazebo reference="left_wheel">
+    <mu1>1.0</mu1>
+    <mu2>0.5</mu2>
+    <material>Gazebo/Black</material>
+  </gazebo>
+  <gazebo reference="right_wheel">
+    <mu1>1.0</mu1>
+    <mu2>0.5</mu2>
+    <material>Gazebo/Black</material>
+  </gazebo>
 <gazebo>
   <plugin name="differential_drive_controller" filename="libgazebo_ros_diff_drive.so">
@@ -339,5 +353,5 @@
     <wheelSeparation>0.35</wheelSeparation>
     <wheelDiameter>0.15</wheelDiameter>
-    <torque>1.41</torque>
+    <torque>10</torque>
     <commandTopic>cmd_vel</commandTopic>
     <odometryTopic>odom</odometryTopic>
@@ -393,5 +407,5 @@
       <update_rate>30.0</update_rate>
       <camera name="head">
-        <horizontal_fov>1.3962634</horizontal_fov>
+        <horizontal_fov>1.8</horizontal_fov>
         <image>
           <width>640</width>

Commit message: add laser scanner and fix multi-CNN model

File: dql_robot/urdf/predator.urdf.xacro (robot description, xacro)
@@ -69,5 +69,5 @@
   <joint name="camera_joint1" type="fixed">
     <axis xyz="0 1 0" />
-    <origin xyz="0.2 0.1 0.25" rpy="0 0 0"/>
+    <origin xyz="0.15 0.1 0.25" rpy="0 0 0.3"/>
     <parent link="base_link"/>
     <child link="camera_link1"/>
@@ -75,5 +75,5 @@
   <joint name="camera_joint2" type="fixed">
     <axis xyz="0 1 0" />
-    <origin xyz="0.2 -0.1 0.25" rpy="0 0 0"/>
+    <origin xyz="0.15 -0.1 0.25" rpy="0 0 -0.3"/>
     <parent link="base_link"/>
     <child link="camera_link2"/>
@@ -230,4 +230,30 @@
         </friction>
       </surface>
+  </link>
+   <joint name="hokuyo_joint" type="fixed">
+    <axis xyz="0 1 0" />
+    <origin xyz="0.15 0 0.2" rpy="0 0 0"/>
+    <parent link="base_link"/>
+    <child link="hokuyo_link"/>
+  </joint>
+  <!-- Hokuyo Laser -->
+  <link name="hokuyo_link">
+    <collision>
+      <origin xyz="0 0 0" rpy="0 0 0"/>
+      <geometry>
+    <box size="0.1 0.1 0.1"/>
+      </geometry>
+    </collision>
+    <visual>
+      <origin xyz="0 0 0" rpy="0 0 0"/>
+      <geometry>
+        <mesh filename="package://dql_robot/urdf/hokuyo.dae"/>
+      </geometry>
+    </visual>
+    <inertial>
+      <mass value="1e-5" />
+      <origin xyz="0 0 0" rpy="0 0 0"/>
+      <inertia ixx="1e-6" ixy="0" ixz="0" iyy="1e-6" iyz="0" izz="1e-6" />
+    </inertial>
   </link>
   <joint name="base_link_back_wheel1" type="continuous">
@@ -436,4 +462,40 @@
     </sensor>
   </gazebo>
+   <gazebo reference="hokuyo_link">
+    <sensor type="gpu_ray" name="head_hokuyo_sensor">
+      <pose>0 0 0 0 0 0</pose>
+      <visualize>false</visualize>
+      <update_rate>30</update_rate>
+      <ray>
+        <scan>
+          <horizontal>
+            <samples>720</samples>
+            <resolution>1</resolution>
+            <min_angle>-1.570796</min_angle>
+            <max_angle>1.570796</max_angle>
+          </horizontal>
+        </scan>
+        <range>
+          <min>0.10</min>
+          <max>4.0</max>
+          <resolution>0.01</resolution>
+        </range>
+        <noise>
+          <type>gaussian</type>
+          <!-- Noise parameters based on published spec for Hokuyo laser
+               achieving "+-30mm" accuracy at range < 10m.  A mean of 0.0m and
+               stddev of 0.01m will put 99.7% of samples within 0.03m of the true
+               reading. -->
+          <mean>0.0</mean>
+          <stddev>0.01</stddev>
+        </noise>
+      </ray>
+      <plugin name="gazebo_ros_head_hokuyo_controller" filename="libgazebo_ros_gpu_laser.so">
+        <topicName>scan</topicName>
+        <frameName>hokuyo_link</frameName>
+      </plugin>
+    </sensor>
+  </gazebo>
+  <xacro:property name="hokuyo_link" value="0.05" />
   <xacro:property name="camera_link1" value="0.05" /> <!-- Size of square 'camera' box -->
   <xacro:property name="camera_link2" value="0.05" /> <!-- Size of square 'camera' box -->

File: dql_robot/urdf/prey.urdf.xacro (robot description, xacro)
@@ -249,4 +249,30 @@
     <origin xyz="-0.15 -0.1 0.025"/>
   </joint>
+   <joint name="hokuyo_joint" type="fixed">
+    <axis xyz="0 1 0" />
+    <origin xyz="0.15 0 0.2" rpy="0 0 0"/>
+    <parent link="base_link"/>
+    <child link="hokuyo_link"/>
+  </joint>
+  <!-- Hokuyo Laser -->
+  <link name="hokuyo_link">
+    <collision>
+      <origin xyz="0 0 0" rpy="0 0 0"/>
+      <geometry>
+    <box size="0.1 0.1 0.1"/>
+      </geometry>
+    </collision>
+    <visual>
+      <origin xyz="0 0 0" rpy="0 0 0"/>
+      <geometry>
+        <mesh filename="package://dql_robot/urdf/hokuyo.dae"/>
+      </geometry>
+    </visual>
+    <inertial>
+      <mass value="1e-5" />
+      <origin xyz="0 0 0" rpy="0 0 0"/>
+      <inertia ixx="1e-6" ixy="0" ixz="0" iyy="1e-6" iyz="0" izz="1e-6" />
+    </inertial>
+  </link>
   <!--link name="right_back_wheel">
   <inertial>
@@ -442,4 +468,40 @@
     </sensor>
   </gazebo>
+    <gazebo reference="hokuyo_link">
+    <sensor type="gpu_ray" name="head_hokuyo_sensor">
+      <pose>0 0 0 0 0 0</pose>
+      <visualize>false</visualize>
+      <update_rate>30</update_rate>
+      <ray>
+        <scan>
+          <horizontal>
+            <samples>720</samples>
+            <resolution>1</resolution>
+            <min_angle>-1.570796</min_angle>
+            <max_angle>1.570796</max_angle>
+          </horizontal>
+        </scan>
+        <range>
+          <min>0.10</min>
+          <max>4.0</max>
+          <resolution>0.01</resolution>
+        </range>
+        <noise>
+          <type>gaussian</type>
+          <!-- Noise parameters based on published spec for Hokuyo laser
+               achieving "+-30mm" accuracy at range < 10m.  A mean of 0.0m and
+               stddev of 0.01m will put 99.7% of samples within 0.03m of the true
+               reading. -->
+          <mean>0.0</mean>
+          <stddev>0.01</stddev>
+        </noise>
+      </ray>
+      <plugin name="gazebo_ros_head_hokuyo_controller" filename="libgazebo_ros_gpu_laser.so">
+        <topicName>scan</topicName>
+        <frameName>hokuyo_link</frameName>
+      </plugin>
+    </sensor>
+  </gazebo>
+  <xacro:property name="hokuyo_link" value="0.05" />
   <xacro:property name="camera_link1" value="0.05" /> <!-- Size of square 'camera' box -->
   <xacro:property name="camera_link2" value="0.05" /> <!-- Size of square 'camera' box -->

Commit message: or

File: dql_robot/urdf/predator.urdf.xacro (robot description, xacro)
@@ -47,35 +47,9 @@
     </inertial>
   </link>
-  <link name="camera_link2">
-    <collision>
-      <origin xyz="0 0 0" rpy="0 0 0"/>
-      <geometry>
-    <box size="0.01 0.01 0.01"/>
-      </geometry>
-    </collision>
-    <visual>
-      <origin xyz="0 0 0" rpy="0 0 0"/>
-      <geometry>
-    <box size="0.01 0.01 0.01"/>
-      </geometry>
-      <material name="red"/>
-    </visual>
-    <inertial>
-      <mass value="1e-5" />
-      <origin xyz="0 0 0" rpy="0 0 0"/>
-      <inertia ixx="1e-6" ixy="0" ixz="0" iyy="1e-6" iyz="0" izz="1e-6" />
-    </inertial>
-  </link>
   <joint name="camera_joint1" type="fixed">
     <axis xyz="0 1 0" />
-    <origin xyz="0.15 0.1 0.25" rpy="0 0 0.3"/>
+    <origin xyz="0.15 0.0 0.25" rpy="0 0 0"/>
     <parent link="base_link"/>
     <child link="camera_link1"/>
-  </joint>
-  <joint name="camera_joint2" type="fixed">
-    <axis xyz="0 1 0" />
-    <origin xyz="0.15 -0.1 0.25" rpy="0 0 -0.3"/>
-    <parent link="base_link"/>
-    <child link="camera_link2"/>
   </joint>
   <link name="box">
@@ -387,5 +361,5 @@
       <update_rate>30.0</update_rate>
       <camera name="head">
-        <horizontal_fov>1.3</horizontal_fov>
+        <horizontal_fov>2.2</horizontal_fov>
         <image>
           <width>640</width>
@@ -409,5 +383,5 @@
         <alwaysOn>true</alwaysOn>
         <updateRate>0.0</updateRate>
-        <cameraName>/right_camera</cameraName>
+        <cameraName>/camera</cameraName>
         <imageTopicName>image_raw</imageTopicName>
         <cameraInfoTopicName>camera_info</cameraInfoTopicName>
@@ -422,48 +396,8 @@
     </sensor>
   </gazebo>
-	<!-- back camera -->
-  <gazebo reference="camera_link2">
-    <sensor type="camera" name="camera2">
-      <update_rate>30.0</update_rate>
-      <camera name="head">
-        <horizontal_fov>1.3</horizontal_fov>
-        <image>
-          <width>640</width>
-          <height>480</height>
-          <format>R8G8B8</format>
-        </image>
-        <clip>
-          <near>0.02</near>
-          <far>300</far>
-        </clip>
-        <noise>
-          <type>gaussian</type>
-          <!-- Noise is sampled independently per pixel on each frame.
-               That pixel's noise value is added to each of its color
-               channels, which at that point lie in the range [0,1]. -->
-          <mean>0.0</mean>
-          <stddev>0.007</stddev>
-        </noise>
-      </camera>
-      <plugin name="camera_controller" filename="libgazebo_ros_camera.so">
-        <alwaysOn>true</alwaysOn>
-        <updateRate>0.0</updateRate>
-        <cameraName>/left_camera</cameraName>
-        <imageTopicName>image_raw</imageTopicName>
-        <cameraInfoTopicName>camera_info</cameraInfoTopicName>
-        <frameName>camera_link2</frameName>
-        <hackBaseline>0.07</hackBaseline>
-        <distortionK1>0.0</distortionK1>
-        <distortionK2>0.0</distortionK2>
-        <distortionK3>0.0</distortionK3>
-        <distortionT1>0.0</distortionT1>
-        <distortionT2>0.0</distortionT2>
-      </plugin>
-    </sensor>
-  </gazebo>
    <gazebo reference="hokuyo_link">
     <sensor type="gpu_ray" name="head_hokuyo_sensor">
       <pose>0 0 0 0 0 0</pose>
-      <visualize>true</visualize>
+      <visualize>false</visualize>
       <update_rate>30</update_rate>
       <ray>
@@ -478,5 +412,5 @@
         <range>
           <min>0.10</min>
-          <max>30.0</max>
+          <max>10.0</max>
           <resolution>0.01</resolution>
         </range>

File: dql_robot/urdf/prey.urdf.xacro (robot description, xacro)
@@ -433,5 +433,5 @@
       <update_rate>30.0</update_rate>
       <camera name="head">
-        <horizontal_fov>1.8</horizontal_fov>
+        <horizontal_fov>2.4</horizontal_fov>
         <image>
           <width>640</width>
@@ -471,5 +471,5 @@
     <sensor type="gpu_ray" name="head_hokuyo_sensor">
       <pose>0 0 0 0 0 0</pose>
-      <visualize>true</visualize>
+      <visualize>false</visualize>
       <update_rate>30</update_rate>
       <ray>
@@ -484,5 +484,5 @@
         <range>
           <min>0.10</min>
-          <max>30.0</max>
+          <max>10.0</max>
           <resolution>0.01</resolution>
         </range>
